File: leds_et_motor.sch (EAGLE design)
At the start: 10 parts, among them IC1 74LS595N, IC2 74LS595N

Commit message: updated schematic to correspond with reality
Connections:
- removed net N$30: JP1.1
- removed net N$31: JP1.3
- removed net N$32: JP1.5
- removed net N$33: JP1.7
- removed net N$34: JP1.9
- removed net N$35: JP1.11
- removed net N$36: JP1.13
- removed net N$37: JP1.15
- removed net N$38: JP2.1
- removed net N$39: JP2.3
- removed net N$40: JP2.5
- removed net N$41: JP2.7
- removed net N$42: JP2.9
- removed net N$43: JP2.11
- removed net N$44: JP2.13
- removed net N$45: JP2.15
- net LED0: now also JP1.15
- net LED1: now also JP1.1
- net LED10: now also JP2.3
- net LED11: now also JP2.5
- net LED12: now also JP2.7
- net LED13: now also JP2.9
- net LED14: now also JP2.11
- net LED15: now also JP2.13
- net LED2: now also JP1.3
- net LED3: now also JP1.5
- net LED4: now also JP1.7
- net LED5: now also JP1.9
- net LED6: now also JP1.11
- net LED7: now also JP1.13
- net LED8: now also JP2.15
- net LED9: now also JP2.1
Other:
- note added: "Arduino pins: 3,5,6,9,10 Pin 9 is currently motor control and connected to PWM_IN1"
- note added: "Strictly speaking I think the even pins are the "top" or "inner" ones so if making a proper board you may need to swap these"
- note removed: "Arduino pins: 3,5,6,9,10"
- note removed: "TODO: mark the QA output to correct pin (forgot to shift the 595s by one...)"
Changed lines of the file:
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@@
 CLK = 13
 MOSI = 11</text>
-<text x="-15.24" y="104.14" size="1.778" layer="97">Arduino pins:
-3,5,6,9,10</text>
-<text x="78.74" y="17.78" size="1.778" layer="97">TODO: mark the QA output to correct pin
-(forgot to shift the 595s by one...) </text>
+<text x="-17.78" y="83.82" size="1.778" layer="97">Arduino pins:
+3,5,6,9,10
+Pin 9 is currently motor control
+and connected to PWM_IN1</text>
 <text x="25.4" y="119.38" size="1.778" layer="97">TODO: LED13-15 signals are not wired to the darlington
 right now, will maybe do it later if it's needed.</text>
+<text x="104.14" y="60.96" size="1.778" layer="97">Strictly speaking I think the even pins
+are the "top" or "inner" ones
+so if making a proper board
+you may need to swap these</text>
 </plain>
 <instances>
@@
 <label x="71.12" y="50.8" size="1.778" layer="95"/>
 </segment>
+<segment>
+<pinref part="JP1" gate="A" pin="15"/>
+<wire x1="114.3" y1="33.02" x2="106.68" y2="33.02" width="0.1524" layer="91"/>
+<label x="99.06" y="33.02" size="1.778" layer="95"/>
+</segment>
 </net>
 <net name="LED7" class="0">
@@
 <label x="71.12" y="33.02" size="1.778" layer="95"/>
 </segment>
+<segment>
+<pinref part="JP1" gate="A" pin="13"/>
+<wire x1="114.3" y1="35.56" x2="106.68" y2="35.56" width="0.1524" layer="91"/>
+<label x="99.06" y="35.56" size="1.778" layer="95"/>
+</segment>
 </net>
 <net name="LED6" class="0">
@@
 <label x="71.12" y="35.56" size="1.778" layer="95"/>
 </segment>
+<segment>
+<pinref part="JP1" gate="A" pin="11"/>
+<wire x1="114.3" y1="38.1" x2="106.68" y2="38.1" width="0.1524" layer="91"/>
+<label x="99.06" y="38.1" size="1.778" layer="95"/>
+</segment>
 </net>
 <net name="LED1" class="0">
@@
 <label x="71.12" y="48.26" size="1.778" layer="95"/>
 </segment>
+<segment>
+<pinref part="JP1" gate="A" pin="1"/>
+<wire x1="114.3" y1="50.8" x2="106.68" y2="50.8" width="0.1524" layer="91"/>
+<label x="99.06" y="50.8" size="1.778" layer="95"/>
+</segment>
 </net>
 <net name="LED2" class="0">
@@
 <label x="71.12" y="45.72" size="1.778" layer="95"/>
 </segment>
+<segment>
+<pinref part="JP1" gate="A" pin="3"/>
+<wire x1="114.3" y1="48.26" x2="106.68" y2="48.26" width="0.1524" layer="91"/>
+<label x="99.06" y="48.26" size="1.778" layer="95"/>
+</segment>
 </net>
 <net name="LED3" class="0">
@@
 <label x="71.12" y="43.18" size="1.778" layer="95"/>
 </segment>
+<segment>
+<pinref part="JP1" gate="A" pin="5"/>
+<wire x1="114.3" y1="45.72" x2="106.68" y2="45.72" width="0.1524" layer="91"/>
+<label x="99.06" y="45.72" size="1.778" layer="95"/>
+</segment>
 </net>
 <net name="LED4" class="0">
@@
 <label x="71.12" y="40.64" size="1.778" layer="95"/>
 </segment>
+<segment>
+<pinref part="JP1" gate="A" pin="7"/>
+<wire x1="114.3" y1="43.18" x2="106.68" y2="43.18" width="0.1524" layer="91"/>
+<label x="99.06" y="43.18" size="1.778" layer="95"/>
+</segment>
 </net>
 <net name="LED5" class="0">
@@
 <wire x1="66.04" y1="38.1" x2="71.12" y2="38.1" width="0.1524" layer="91"/>
 <label x="71.12" y="38.1" size="1.778" layer="95"/>
+</segment>
+<segment>
+<pinref part="JP1" gate="A" pin="9"/>
+<wire x1="114.3" y1="40.64" x2="106.68" y2="40.64" width="0.1524" layer="91"/>
+<label x="99.06" y="40.64" size="1.778" layer="95"/>
 </segment>
 </net>
@@
 <label x="71.12" y="10.16" size="1.778" layer="95"/>
 </segment>
+<segment>
+<pinref part="JP2" gate="A" pin="15"/>
+<wire x1="114.3" y1="-7.62" x2="106.68" y2="-7.62" width="0.1524" layer="91"/>
+<label x="99.06" y="-7.62" size="1.778" layer="95"/>
+</segment>
 </net>
 <net name="LED9" class="0">
@@
 <label x="71.12" y="7.62" size="1.778" layer="95"/>
 </segment>
+<segment>
+<pinref part="JP2" gate="A" pin="1"/>
+<wire x1="114.3" y1="10.16" x2="106.68" y2="10.16" width="0.1524" layer="91"/>
+<label x="99.06" y="10.16" size="1.778" layer="95"/>
+</segment>
 </net>
 <net name="LED10" class="0">
@@
 <label x="71.12" y="5.08" size="1.778" layer="95"/>
 </segment>
+<segment>
+<pinref part="JP2" gate="A" pin="3"/>
+<wire x1="114.3" y1="7.62" x2="106.68" y2="7.62" width="0.1524" layer="91"/>
+<label x="99.06" y="7.62" size="1.778" layer="95"/>
+</segment>
 </net>
 <net name="LED11" class="0">
@@
 <label x="71.12" y="2.54" size="1.778" layer="95"/>
 </segment>
+<segment>
+<pinref part="JP2" gate="A" pin="5"/>
+<wire x1="114.3" y1="5.08" x2="106.68" y2="5.08" width="0.1524" layer="91"/>
+<label x="99.06" y="5.08" size="1.778" layer="95"/>
+</segment>
 </net>
 <net name="LED12" class="0">
@@
 <label x="71.12" y="0" size="1.778" layer="95"/>
 </segment>
+<segment>
+<pinref part="JP2" gate="A" pin="7"/>
+<wire x1="114.3" y1="2.54" x2="106.68" y2="2.54" width="0.1524" layer="91"/>
+<label x="99.06" y="2.54" size="1.778" layer="95"/>
+</segment>
 </net>
 <net name="LED13" class="0">
@@
 <label x="38.1" y="111.76" size="1.778" layer="95"/>
 </segment>
+<segment>
+<pinref part="JP2" gate="A" pin="9"/>
+<wire x1="114.3" y1="0" x2="106.68" y2="0" width="0.1524" layer="91"/>
+<label x="99.06" y="0" size="1.778" layer="95"/>
+</segment>
 </net>
 <net name="LED14" class="0">
@@
 <label x="38.1" y="106.68" size="1.778" layer="95"/>
 </segment>
+<segment>
+<pinref part="JP2" gate="A" pin="11"/>
+<wire x1="114.3" y1="-2.54" x2="106.68" y2="-2.54" width="0.1524" layer="91"/>
+<label x="99.06" y="-2.54" size="1.778" layer="95"/>
+</segment>
 </net>
 <net name="LED15" class="0">
@@
 <wire x1="50.8" y1="101.6" x2="45.72" y2="101.6" width="0.1524" layer="91"/>
 <label x="38.1" y="101.6" size="1.778" layer="95"/>
+</segment>
+<segment>
+<pinref part="JP2" gate="A" pin="13"/>
+<wire x1="114.3" y1="-5.08" x2="106.68" y2="-5.08" width="0.1524" layer="91"/>
+<label x="99.06" y="-5.08" size="1.778" layer="95"/>
 </segment>
 </net>
@@
 </segment>
 </net>
-<net name="N$30" class="0">
-<segment>
-<pinref part="JP1" gate="A" pin="1"/>
-<wire x1="114.3" y1="50.8" x2="106.68" y2="50.8" width="0.1524" layer="91"/>
-</segment>
-</net>
-<net name="N$31" class="0">
-<segment>
-<pinref part="JP1" gate="A" pin="3"/>
-<wire x1="114.3" y1="48.26" x2="106.68" y2="48.26" width="0.1524" layer="91"/>
-</segment>
-</net>
-<net name="N$32" class="0">
-<segment>
-<pinref part="JP1" gate="A" pin="5"/>
-<wire x1="114.3" y1="45.72" x2="106.68" y2="45.72" width="0.1524" layer="91"/>
-</segment>
-</net>
-<net name="N$33" class="0">
-<segment>
-<pinref part="JP1" gate="A" pin="7"/>
-<wire x1="114.3" y1="43.18" x2="106.68" y2="43.18" width="0.1524" layer="91"/>
-</segment>
-</net>
-<net name="N$34" class="0">
-<segment>
-<pinref part="JP1" gate="A" pin="9"/>
-<wire x1="114.3" y1="40.64" x2="106.68" y2="40.64" width="0.1524" layer="91"/>
-</segment>
-</net>
-<net name="N$35" class="0">
-<segment>
-<pinref part="JP1" gate="A" pin="11"/>
-<wire x1="114.3" y1="38.1" x2="106.68" y2="38.1" width="0.1524" layer="91"/>
-</segment>
-</net>
-<net name="N$36" class="0">
-<segment>
-<pinref part="JP1" gate="A" pin="13"/>
-<wire x1="114.3" y1="35.56" x2="106.68" y2="35.56" width="0.1524" layer="91"/>
-</segment>
-</net>
-<net name="N$37" class="0">
-<segment>
-<pinref part="JP1" gate="A" pin="15"/>
-<wire x1="114.3" y1="33.02" x2="106.68" y2="33.02" width="0.1524" layer="91"/>
-</segment>
-</net>
-<net name="N$38" class="0">
-<segment>
-<pinref part="JP2" gate="A" pin="1"/>
-<wire x1="114.3" y1="10.16" x2="106.68" y2="10.16" width="0.1524" layer="91"/>
-</segment>
-</net>
-<net name="N$39" class="0">
-<segment>
-<pinref part="JP2" gate="A" pin="3"/>
-<wire x1="114.3" y1="7.62" x2="106.68" y2="7.62" width="0.1524" layer="91"/>
-</segment>
-</net>
-<net name="N$40" class="0">
-<segment>
-<pinref part="JP2" gate="A" pin="5"/>
-<wire x1="114.3" y1="5.08" x2="106.68" y2="5.08" width="0.1524" layer="91"/>
-</segment>
-</net>
-<net name="N$41" class="0">
-<segment>
-<pinref part="JP2" gate="A" pin="7"/>
-<wire x1="114.3" y1="2.54" x2="106.68" y2="2.54" width="0.1524" layer="91"/>
-</segment>
-</net>
-<net name="N$42" class="0">
-<segment>
-<pinref part="JP2" gate="A" pin="9"/>
-<wire x1="114.3" y1="0" x2="106.68" y2="0" width="0.1524" layer="91"/>
-</segment>
-</net>
-<net name="N$43" class="0">
-<segment>
-<pinref part="JP2" gate="A" pin="11"/>
-<wire x1="114.3" y1="-2.54" x2="106.68" y2="-2.54" width="0.1524" layer="91"/>
-</segment>
-</net>
-<net name="N$44" class="0">
-<segment>
-<pinref part="JP2" gate="A" pin="13"/>
-<wire x1="114.3" y1="-5.08" x2="106.68" y2="-5.08" width="0.1524" layer="91"/>
-</segment>
-</net>
-<net name="N$45" class="0">
-<segment>
-<pinref part="JP2" gate="A" pin="15"/>
-<wire x1="114.3" y1="-7.62" x2="106.68" y2="-7.62" width="0.1524" layer="91"/>
-</segment>
-</net>

Commit message: some notes
Other:
- note added: "12V goes to Vin GNDs to GNDs 5V to 5V"
- note added: "Bypass caps not drawn (also actually forgot to add them to the veroboard, it works anyway)"
- note added: "Main 12V input There is switch on the +12V on the incoming line"
Changed lines of the file:
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@@
 so if making a proper board
 you may need to swap these</text>
+<text x="-20.32" y="35.56" size="1.778" layer="97">12V goes to Vin
+GNDs to GNDs
+5V to 5V</text>
+<text x="-30.48" y="5.08" size="1.778" layer="97">Main 12V input
+There is switch on the +12V
+on the incoming line</text>
+<text x="33.02" y="-25.4" size="1.778" layer="97">Bypass caps not drawn
+(also actually forgot to add them to
+the veroboard, it works anyway)</text>
 </plain>
 <instances>
